Commit message: feat : sungnam 지도 작성, ugv_model base_footprint 수정

File: urdf/ugv_model.urdf (robot description, URDF)
Before this commit: robot HAS-UGV, 7 links, 6 joints
Links:
- added link base_footprint, mass 0.001; visual box size=0.001 0.001 0.0011
Joints:
- added joint base_footprint_joint: type fixed, parent base_footprint, child base_link, origin xyz=0.45 0 0.4435 rpy=0 0 -1.58
- joint base_laser_tower_to_laser: origin xyz=0 0 0 -> xyz=0 0 0.15 rpy=0 0 1.5708
- joint base_link_joint: origin xyz=0 0 0 -> xyz=0 0.382 0.4485
- joint base_to_wheel1: origin xyz=0 0 0 -> xyz=0.56 0.723 -0.1361
- joint base_to_wheel2: origin xyz=0 0 0 -> xyz=-0.56 0.723 -0.1361
- joint base_to_wheel3: origin xyz=0 0 0 -> xyz=0.56 -0.723 -0.1361
- joint base_to_wheel4: origin xyz=0 0 0 -> xyz=-0.56 -0.723 -0.1361

Commit message: feat : urdf 로봇 가로 세로 변경

File: urdf/ugv_model.urdf (robot description, URDF)
Before this commit: robot HAS-UGV, 8 links, 7 joints
Links:
- link base_link: geometry collision box size=1.998 1.12 0.677; visual box size=1.998 1.12 0.677
Joints:
- joint base_footprint_joint: origin xyz=0.45 0 0.4435 rpy=0 0 -1.58 -> xyz=0.0 0 0.4435 rpy=0 0 0
- joint base_laser_tower_to_laser: origin xyz=0 0 0.15 rpy=0 0 1.5708 -> xyz=0 0 0.15 rpy=0 0 0
- joint base_link_joint: origin xyz=0 0.382 0.4485 -> xyz=0.832 0 0.4485
- joint base_to_wheel1: origin xyz=0.56 0.723 -0.1361 -> xyz=1.173 0.56 -0.1361 rpy=0 0 1.57
- joint base_to_wheel2: origin xyz=-0.56 0.723 -0.1361 -> xyz=1.173 -0.56 -0.1361 rpy=0 0 1.57
- joint base_to_wheel3: origin xyz=0.56 -0.723 -0.1361 -> xyz=-0.273 0.56 -0.1361 rpy=0 0 1.57
- joint base_to_wheel4: origin xyz=-0.56 -0.723 -0.1361 -> xyz=-0.273 -0.56 -0.1361 rpy=0 0 1.57

Commit message: feat : ugv_model - sick lidar front, back to add urdf

File: urdf/ugv_model.urdf (robot description, URDF)
Before this commit: robot HAS-UGV, 8 links, 7 joints
Links:
- added link back_laser_link, mass 0.00001; visual cylinder length=0.085 radius=0.076
- added link front_laser_link, mass 0.00001; visual cylinder length=0.085 radius=0.076
Joints:
- added joint base_link_to_back_laser_link: type fixed, parent base_link, child back_laser_link, origin xyz=-0.549 0 0 rpy=0 0 3.14
- added joint base_link_to_front_laser_link: type fixed, parent base_link, child front_laser_link, origin xyz=1.449 0 0

Commit message: feat : log Add

File: urdf/ugv_model.urdf (robot description, URDF)
Before this commit: robot HAS-UGV, 8 links, 7 joints
Links:
- added link back_laser_link, mass 0.00001; visual cylinder length=0.085 radius=0.076
- added link front_laser_link, mass 0.00001; visual cylinder length=0.085 radius=0.076
- link base_link: geometry collision box size=1.998 1.12 0.677; visual box size=1.998 1.12 0.677
Joints:
- added joint base_link_to_back_laser_link: type fixed, parent base_link, child back_laser_link, origin xyz=-0.549 0 0
- added joint base_link_to_front_laser_link: type fixed, parent base_link, child front_laser_link, origin xyz=1.449 0 0
- joint base_footprint_joint: origin xyz=0.45 0 0.4435 rpy=0 0 -1.58 -> xyz=0.0 0 0.4435 rpy=0 0 0
- joint base_laser_tower_to_laser: origin xyz=0 0 0.15 rpy=0 0 1.5708 -> xyz=0 0 0.15 rpy=0 0 0
- joint base_link_joint: origin xyz=0 0.382 0.4485 -> xyz=0.832 0 0.4485
- joint base_to_wheel1: origin xyz=0.56 0.723 -0.1361 -> xyz=1.173 0.56 -0.1361 rpy=0 0 1.57
- joint base_to_wheel2: origin xyz=-0.56 0.723 -0.1361 -> xyz=1.173 -0.56 -0.1361 rpy=0 0 1.57
- joint base_to_wheel3: origin xyz=0.56 -0.723 -0.1361 -> xyz=-0.273 0.56 -0.1361 rpy=0 0 1.57
- joint base_to_wheel4: origin xyz=-0.56 -0.723 -0.1361 -> xyz=-0.273 -0.56 -0.1361 rpy=0 0 1.57
