Commit message: feat : wkvalve_test upload

File: urdf/atc_model.urdf (robot description, URDF)
Before this commit: robot HAS-UGV, 9 links, 8 joints
Joints:
- joint base_link_to_back_laser_link: origin xyz=-0.5 0 0 -> xyz=-0.5 0 0 rpy=0 0 3.14

File: urdf/ugv_model.urdf (robot description, URDF)
Before this commit: robot HAS-UGV, 10 links, 9 joints
Joints:
- joint base_link_to_back_laser_link: origin xyz=-0.549 0 0 rpy=0 0 3.14 -> xyz=-0.549 0 0

Commit message: feat : UGV for ADD docker

File: urdf/atc_model.urdf (robot description, URDF)
Before this commit: robot HAS-UGV, 9 links, 8 joints
Links:
- removed link front_laser_link
- added link base_laser_link, mass 0.00001; visual cylinder length=0.085 radius=0.076
Joints:
- removed joint base_link_to_front_laser_link
- added joint base_link_to_base_laser_link: type fixed, parent base_link, child base_laser_link, origin xyz=1.5 0 0

File: urdf/ugv_model.urdf (robot description, URDF)
Before this commit: robot HAS-UGV, 10 links, 9 joints
Joints:
- joint base_link_to_back_laser_link: origin xyz=-0.549 0 0 -> xyz=-0.549 0 0 rpy=0 0 3.14
